File: Hardware/Receiver/ReceiverE5.sch (KiCad schematic (older format))
At the start: 39 parts, among them J1 KBUS, J2 AVR-PDI-6A, J3 CONN_01X08, J4 CONN_01X06, J5 CONN_01X06, J6 CONN_01X04, J7 CONN_01X04, U1 ATXMEGA32E5-A, U2 LM2731, U3 SN74LV07A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

Commit message: Added some extra fields for BOM generation with kibom
Parts:
- J1: BOM_Footprint (none) -> Type A, TH, FCI 87520
- J3, J4, J5, J6, J7: BOM_Footprint (none) -> no part
Changed lines of the file:
@@
 F 2 "kuro:USB_A_multicomp" V 900 1400 50  0001 C CNN
 F 3 "" V 900 1400 50  0000 C CNN
+F 4 "Type A, TH, FCI 87520" V 950 1500 60  0001 C CNN "BOM_Footprint"
 	1    950  1500
 	0    -1   1    0
@@
 F 2 "Pin_Headers:Pin_Header_Straight_1x08" H 3850 6750 50  0001 C CNN
 F 3 "" H 3850 6750 50  0000 C CNN
+F 4 "no part" H 3850 6750 60  0001 C CNN "BOM_Footprint"
 	1    3850 6750
 	1    0    0    -1
@@
 F 2 "Pin_Headers:Pin_Header_Straight_1x06" H 7600 4000 50  0001 C CNN
 F 3 "" H 7600 4000 50  0000 C CNN
+F 4 "no part" H 7600 4000 60  0001 C CNN "BOM_Footprint"
 	1    7600 4000
 	1    0    0    -1
@@
 F 2 "Pin_Headers:Pin_Header_Straight_1x06" H 7600 4950 50  0001 C CNN
 F 3 "" H 7600 4950 50  0000 C CNN
+F 4 "no part" H 7600 4950 60  0001 C CNN "BOM_Footprint"
 	1    7600 4950
 	1    0    0    -1
@@
 F 2 "Pin_Headers:Pin_Header_Straight_1x04" H 10650 4000 50  0001 C CNN
 F 3 "" H 10650 4000 50  0000 C CNN
+F 4 "no part" H 10650 4000 60  0001 C CNN "BOM_Footprint"
 	1    10650 4000
 	1    0    0    -1
@@
 F 2 "Pin_Headers:Pin_Header_Straight_1x04" H 10650 5700 50  0001 C CNN
 F 3 "" H 10650 5700 50  0000 C CNN
+F 4 "no part" H 10650 5700 60  0001 C CNN "BOM_Footprint"
 	1    10650 5700
 	1    0    0    -1

Commit message: Added BOM + notes
Parts:
- D2: BOM_Note (none) -> 9556915, 463-432
- J1: BOM_Note (none) -> 2112381, 771-0057
- U1: BOM_Note (none) -> 2327713, 899-6912
- U2: BOM_Note (none) -> 1564771, 761-5567
- U3, U4: BOM_Note (none) -> 1774543, 662-8402
- U5: BOM_Note (none) -> 1710835, 709-8758
- U6, U7: BOM_Note (none) -> 2444915, 816-8842
Changed lines of the file:
@@
 F 2 "TO_SOT_Packages_SMD:SOT-23-5" H 4050 1450 100 0001 C CNN
 F 3 "" H 4050 1450 100 0000 C CNN
+F 4 "1564771, 761-5567" H 4050 1450 60  0001 C CNN "BOM_Note"
 	1    4050 1450
 	1    0    0    -1
@@
 F 2 "Diodes_SMD:SOD-123" H 4900 1250 50  0001 C CNN
 F 3 "" H 4900 1250 50  0000 C CNN
+F 4 "9556915, 463-432" H 4900 1250 60  0001 C CNN "BOM_Note"
 	1    4900 1250
 	-1   0    0    1
@@
 F 3 "" V 900 1400 50  0000 C CNN
 F 4 "Type A, TH, FCI 87520" V 950 1500 60  0001 C CNN "BOM_Footprint"
+F 5 "2112381, 771-0057" V 950 1500 60  0001 C CNN "BOM_Note"
 	1    950  1500
 	0    -1   1    0
@@
 F 2 "TO_SOT_Packages_SMD:SOT-23-5" H 7200 1250 50  0001 C CNN
 F 3 "" H 7200 1500 60  0000 C CNN
+F 4 "1710835, 709-8758" H 7200 1500 60  0001 C CNN "BOM_Note"
 	1    7200 1500
 	1    0    0    -1
@@
 F 2 "Housings_QFP:TQFP-32_7x7mm_Pitch0.8mm" H 3850 4550 50  0001 C CIN
 F 3 "" H 3850 4550 50  0000 C CNN
+F 4 "2327713, 899-6912" H 3850 4550 60  0001 C CNN "BOM_Note"
 	1    3850 4550
 	1    0    0    -1
@@
 F 2 "SMD_Packages:SSOP-14" H 6850 4050 100 0001 C CNN
 F 3 "" H 6850 4050 100 0000 C CNN
+F 4 "1774543, 662-8402" H 6850 4050 60  0001 C CNN "BOM_Note"
 	1    6850 4050
 	1    0    0    -1
@@
 F 2 "SMD_Packages:SSOP-14" H 6850 5000 100 0001 C CNN
 F 3 "" H 6850 5000 100 0000 C CNN
+F 4 "1774543, 662-8402" H 6850 5000 60  0001 C CNN "BOM_Note"
 	1    6850 5000
 	1    0    0    -1
@@
 F 2 "kuro:VSSOP8_SOT765-1" H 9100 3900 60  0001 C CNN
 F 3 "" H 9100 3900 60  0000 C CNN
+F 4 "2444915, 816-8842" H 9100 3900 60  0001 C CNN "BOM_Note"
 	1    9100 3900
 	1    0    0    -1
@@
 F 2 "kuro:VSSOP8_SOT765-1" H 9100 4800 60  0001 C CNN
 F 3 "" H 9100 4800 60  0000 C CNN
+F 4 "2444915, 816-8842" H 9100 4800 60  0001 C CNN "BOM_Note"
 	1    9100 4800
 	1    0    0    -1
