File: Hardware/Receiver V2.0/ReceiverE5.sch (KiCad schematic (older format))
At the start: 40 parts, among them J1 KBUS, J2 AVR-PDI-6A, J3 CONN_01X08, J4 CONN_01X06, J5 CONN_01X06, J6 CONN_01X04, J7 CONN_01X04, SW1 SW_SPST, U1 ATXMEGA32E5-A, U2 LM2731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

Commit message: Widened board, added button
Parts:
- removed SW1: SW_SPST, Buttons_Switches_SMD:SW_SPST_EVQP7C, symbol SW_SPST
- D1: symbol LED-RESCUE-ReceiverE5 -> LED
- J1: symbol USB_A-RESCUE-ReceiverE5 -> USB_A
Connections:
- wire segments 214 -> 209
- no-connect marks 2 -> 3
