File: Joystick/hardware/V2.0/_saved_superplay.sch (KiCad schematic (older format))
At the start: 32 parts, among them J1 AVR-PDI-6A, J2 CONN_02X04, J3 USB_B, U1 MCP1700T-3002E, U2 ATXMEGA128A3U-A, U3 TPD4S009DBV, Y1 16MHz

Commit message: Assigned footprints
Parts:
- C1, C10, C11, C3, C4, C5, C6, C7, C8, C9: footprint (none) -> Capacitors_SMD:C_0603
- C2: footprint (none) -> Capacitors_SMD:C_1206
- D1: footprint (none) -> LEDs:LED_0603
- J1: footprint AVR-PDI-6 -> kuro:3x2_1.27mm_SMD_header
- J3: footprint (none) -> Connectors_Molex:USB_Micro-B_Molex_47346-0001
- PA1, PA2, PB1, PB2, PB3, PB4, PJ1, PR1, PR2, PR3: footprint (none) -> kuro:B5B-ZR-SM4-TF
- R1: footprint (none) -> Resistors_SMD:R_0603
- U1: footprint (none) -> TO_SOT_Packages_SMD:SOT-23
- U2: footprint TQFP64 -> Housings_QFP:TQFP-64_14x14mm_Pitch0.8mm
- U3: footprint (none) -> TO_SOT_Packages_SMD:SOT-23-6
