File: Joystick/hardware/V2.0/superplay.sch (KiCad schematic (older format))
At the start: 32 parts, among them J1 AVR-PDI-6A, J2 CONN_02X04, J3 USB_B, U1 MCP1700T-3002E, U2 ATXMEGA128A3U-A, U3 TPD4S009DBV, Y1 16MHz

Commit message: Finished foorprint assignments
Parts:
- C1, C10, C11, C3, C4, C5, C6, C7, C8, C9: footprint (none) -> Capacitors_SMD:C_0603
- C2: footprint (none) -> Capacitors_SMD:C_1206
- D1: footprint (none) -> LEDs:LED_0603
- J1: footprint AVR-PDI-6 -> kuro:3x2_1.27mm_SMD_header
- J2: footprint (none) -> kuro:4x2_1.27mm_SMD_header
- J3: footprint (none) -> Connectors_Molex:USB_Micro-B_Molex_47346-0001
- PA1, PA2, PB1, PB2, PB3, PB4, PJ1, PR1, PR2, PR3: footprint (none) -> kuro:B5B-ZR-SM4-TF
- PL1, PM1: footprint (none) -> kuro:B2B-ZR-SM4-TF
- R1: footprint (none) -> Resistors_SMD:R_0603
- U1: footprint (none) -> TO_SOT_Packages_SMD:SOT-23
- U2: footprint TQFP64 -> Housings_QFP:TQFP-64_14x14mm_Pitch0.8mm
- U3: footprint (none) -> TO_SOT_Packages_SMD:SOT-23-6
- Y1: footprint (none) -> kuro:SMD_Crystal_Multi_QC6CB_7A_ABM7

Commit message: Fixed ERCs
Connections:
- no-connect marks 0 -> 4
Changed lines of the file:
@@
 encoding utf-8
 Sheet 1 1
-Title ""
+Title "SUPERPLAY joystick controller"
 Date ""
-Rev ""
-Comp ""
-Comment1 ""
+Rev "2.0"
+Comp "KEIO"
+Comment1 "Licence: GPL V3"
 Comment2 ""
 Comment3 ""
@@
 F 3 "" H 6600 1300 50  0000 C CNN
 	1    6600 1300
-	1    0    0    -1
-$EndComp
-$Comp
-L PWR_FLAG #FLG03
-U 1 1 59143147
-P 4250 900
-F 0 "#FLG03" H 4250 995 50  0001 C CNN
-F 1 "PWR_FLAG" H 4250 1080 50  0000 C CNN
-F 2 "" H 4250 900 50  0000 C CNN
-F 3 "" H 4250 900 50  0000 C CNN
-	1    4250 900
 	1    0    0    -1
 $EndComp
@@
 $EndComp
 $Comp
-L +5V #PWR04
+L +5V #PWR03
 U 1 1 59143C77
 P 6600 800
-F 0 "#PWR04" H 6600 650 50  0001 C CNN
+F 0 "#PWR03" H 6600 650 50  0001 C CNN
 F 1 "+5V" H 6600 940 50  0000 C CNN
 F 2 "" H 6600 800 50  0000 C CNN
@@
 	6900 850  6600 850
 $Comp
-L +3.3V #PWR05
+L +3.3V #PWR04
 U 1 1 59145907
 P 4200 1600
-F 0 "#PWR05" H 4200 1450 50  0001 C CNN
+F 0 "#PWR04" H 4200 1450 50  0001 C CNN
 F 1 "+3.3V" H 4200 1740 50  0000 C CNN
 F 2 "" H 4200 1600 50  0000 C CNN
@@
 	2000 4850 3450 4850
 $Comp
-L GND #PWR06
+L GND #PWR05
 U 1 1 59147100
 P 4450 5250
-F 0 "#PWR06" H 4450 5000 50  0001 C CNN
+F 0 "#PWR05" H 4450 5000 50  0001 C CNN
 F 1 "GND" H 4450 5100 50  0000 C CNN
 F 2 "" H 4450 5250 50  0000 C CNN
@@
 	2400 5500 2600 5500
 $Comp
-L GND #PWR07
+L GND #PWR06
 U 1 1 59148957
 P 2550 5650
-F 0 "#PWR07" H 2550 5400 50  0001 C CNN
+F 0 "#PWR06" H 2550 5400 50  0001 C CNN
 F 1 "GND" H 2550 5500 50  0000 C CNN
 F 2 "" H 2550 5650 50  0000 C CNN
@@
 $EndComp
 $Comp
-L +5V #PWR08
+L +5V #PWR07
 U 1 1 59148B1C
 P 3650 5550
-F 0 "#PWR08" H 3650 5400 50  0001 C CNN
+F 0 "#PWR07" H 3650 5400 50  0001 C CNN
 F 1 "+5V" H 3650 5690 50  0000 C CNN
 F 2 "" H 3650 5550 50  0000 C CNN
@@
 Connection ~ 2500 4850
 $Comp
-L GND #PWR09
+L GND #PWR08
 U 1 1 59149182
 P 1600 5200
-F 0 "#PWR09" H 1600 4950 50  0001 C CNN
+F 0 "#PWR08" H 1600 4950 50  0001 C CNN
 F 1 "GND" H 1600 5050 50  0000 C CNN
 F 2 "" H 1600 5200 50  0000 C CNN
@@
 $EndComp
 $Comp
-L GND #PWR010
+L GND #PWR09
 U 1 1 591491C0
 P 2050 5000
-F 0 "#PWR010" H 2050 4750 50  0001 C CNN
+F 0 "#PWR09" H 2050 4750 50  0001 C CNN
 F 1 "GND" H 2050 4850 50  0000 C CNN
 F 2 "" H 2050 5000 50  0000 C CNN
@@
 	1600 5150 1600 5200
 $Comp
-L +5V #PWR011
+L +5V #PWR010
 U 1 1 591495A3
 P 2050 4600
-F 0 "#PWR011" H 2050 4450 50  0001 C CNN
+F 0 "#PWR010" H 2050 4450 50  0001 C CNN
 F 1 "+5V" H 2050 4740 50  0000 C CNN
 F 2 "" H 2050 4600 50  0000 C CNN
@@
 $EndComp
 $Comp
-L +5V #PWR012
+L +5V #PWR011
 U 1 1 5914A576
 P 6700 3600
-F 0 "#PWR012" H 6700 3450 50  0001 C CNN
+F 0 "#PWR011" H 6700 3450 50  0001 C CNN
 F 1 "+5V" H 6700 3740 50  0000 C CNN
 F 2 "" H 6700 3600 50  0000 C CNN
@@
 $EndComp
 $Comp
-L +3.3V #PWR013
+L +3.3V #PWR012
 U 1 1 5914A5C9
 P 6900 3600
-F 0 "#PWR013" H 6900 3450 50  0001 C CNN
+F 0 "#PWR012" H 6900 3450 50  0001 C CNN
 F 1 "+3.3V" H 6900 3740 50  0000 C CNN
 F 2 "" H 6900 3600 50  0000 C CNN
@@
 $EndComp
 $Comp
-L GND #PWR014
+L GND #PWR013
 U 1 1 5914A60A
 P 6900 4100
-F 0 "#PWR014" H 6900 3850 50  0001 C CNN
+F 0 "#PWR013" H 6900 3850 50  0001 C CNN
 F 1 "GND" H 6900 3950 50  0000 C CNN
 F 2 "" H 6900 4100 50  0000 C CNN
@@
 	2500 3500 2500 3400
 $Comp
-L GND #PWR015
+L GND #PWR014
 U 1 1 5914D44B
 P 2200 3600
-F 0 "#PWR015" H 2200 3350 50  0001 C CNN
+F 0 "#PWR014" H 2200 3350 50  0001 C CNN
 F 1 "GND" H 2200 3450 50  0000 C CNN
 F 2 "" H 2200 3600 50  0000 C CNN
@@
 	1900 1400 2100 1400
 $Comp
-L GND #PWR016
+L GND #PWR015
 U 1 1 59156687
 P 2950 1650
-F 0 "#PWR016" H 2950 1400 50  0001 C CNN
+F 0 "#PWR015" H 2950 1400 50  0001 C CNN
 F 1 "GND" H 2950 1500 50  0000 C CNN
 F 2 "" H 2950 1650 50  0000 C CNN
@@
 $EndComp
 $Comp
-L +3.3V #PWR017
+L +3.3V #PWR016
 U 1 1 59156796
 P 2950 1350
-F 0 "#PWR017" H 2950 1200 50  0001 C CNN
+F 0 "#PWR016" H 2950 1200 50  0001 C CNN
 F 1 "+3.3V" H 2950 1490 50  0000 C CNN
 F 2 "" H 2950 1350 50  0000 C CNN
@@
 	2950 1600 2950 1650
 $Comp
-L +5V #PWR018
-U 1 1 59157201
-P 4550 900
-F 0 "#PWR018" H 4550 750 50  0001 C CNN
-F 1 "+5V" H 4550 1040 50  0000 C CNN
-F 2 "" H 4550 900 50  0000 C CNN
-F 3 "" H 4550 900 50  0000 C CNN
-	1    4550 900
-	1    0    0    -1
-$EndComp
-$Comp
-L +3.3V #PWR019
-U 1 1 5915743C
-P 5150 900
-F 0 "#PWR019" H 5150 750 50  0001 C CNN
-F 1 "+3.3V" H 5150 1040 50  0000 C CNN
-F 2 "" H 5150 900 50  0000 C CNN
-F 3 "" H 5150 900 50  0000 C CNN
-	1    5150 900
-	1    0    0    -1
-$EndComp
-$Comp
-L GND #PWR020
+L GND #PWR017
 U 1 1 59157483
 P 5500 950
-F 0 "#PWR020" H 5500 700 50  0001 C CNN
+F 0 "#PWR017" H 5500 700 50  0001 C CNN
 F 1 "GND" H 5500 800 50  0000 C CNN
 F 2 "" H 5500 950 50  0000 C CNN
@@
 	1    0    0    -1
 $EndComp
-Wire Wire Line
-	4250 900  4250 950
-Wire Wire Line
-	4250 950  4550 950
-Wire Wire Line
-	4550 950  4550 900
-$Comp
-L PWR_FLAG #FLG021
-U 1 1 59158ACD
-P 4850 900
-F 0 "#FLG021" H 4850 995 50  0001 C CNN
-F 1 "PWR_FLAG" H 4850 1080 50  0000 C CNN
-F 2 "" H 4850 900 50  0000 C CNN
-F 3 "" H 4850 900 50  0000 C CNN
-	1    4850 900
-	1    0    0    -1
-$EndComp
-Wire Wire Line
-	4850 900  4850 950
-Wire Wire Line
-	4850 950  5150 950
-Wire Wire Line
-	5150 950  5150 900
-$Comp
-L PWR_FLAG #FLG022
+$Comp
+L PWR_FLAG #FLG018
 U 1 1 59158EEC
 P 5500 900
-F 0 "#FLG022" H 5500 995 50  0001 C CNN
+F 0 "#FLG018" H 5500 995 50  0001 C CNN
 F 1 "PWR_FLAG" H 5500 1080 50  0000 C CNN
 F 2 "" H 5500 900 50  0000 C CNN
@@
 RIGHT
 $Comp
-L GND #PWR023
+L GND #PWR019
 U 1 1 5915A82C
 P 9000 2350
-F 0 "#PWR023" H 9000 2100 50  0001 C CNN
+F 0 "#PWR019" H 9000 2100 50  0001 C CNN
 F 1 "GND" H 9000 2200 50  0000 C CNN
 F 2 "" H 9000 2350 50  0000 C CNN
@@
 	9200 3100 9000 3100
 $Comp
-L GND #PWR024
+L GND #PWR020
 U 1 1 5915BE0E
 P 9000 3150
-F 0 "#PWR024" H 9000 2900 50  0001 C CNN
+F 0 "#PWR020" H 9000 2900 50  0001 C CNN
 F 1 "GND" H 9000 3000 50  0000 C CNN
 F 2 "" H 9000 3150 50  0000 C CNN
@@
 	9000 3900 9200 3900
 $Comp
-L GND #PWR025
+L GND #PWR021
 U 1 1 5915C6F7
 P 9000 3950
-F 0 "#PWR025" H 9000 3700 50  0001 C CNN
+F 0 "#PWR021" H 9000 3700 50  0001 C CNN
 F 1 "GND" H 9000 3800 50  0000 C CNN
 F 2 "" H 9000 3950 50  0000 C CNN
@@
 	9200 4700 9000 4700
 $Comp
-L GND #PWR026
+L GND #PWR022
 U 1 1 5915D6FA
 P 9000 4750
-F 0 "#PWR026" H 9000 4500 50  0001 C CNN
+F 0 "#PWR022" H 9000 4500 50  0001 C CNN
 F 1 "GND" H 9000 4600 50  0000 C CNN
 F 2 "" H 9000 4750 50  0000 C CNN
@@
 	9200 5500 9000 5500
 $Comp
-L GND #PWR027
+L GND #PWR023
 U 1 1 5915DD1D
 P 9000 5550
-F 0 "#PWR027" H 9000 5300 50  0001 C CNN
+F 0 "#PWR023" H 9000 5300 50  0001 C CNN
 F 1 "GND" H 9000 5400 50  0000 C CNN
 F 2 "" H 9000 5550 50  0000 C CNN
@@
 	10350 2300 10150 2300
 $Comp
-L GND #PWR028
+L GND #PWR024
 U 1 1 5915EC68
 P 10150 2350
-F 0 "#PWR028" H 10150 2100 50  0001 C CNN
+F 0 "#PWR024" H 10150 2100 50  0001 C CNN
 F 1 "GND" H 10150 2200 50  0000 C CNN
 F 2 "" H 10150 2350 50  0000 C CNN
@@
 	10350 3100 10150 3100
 $Comp
-L GND #PWR029
+L GND #PWR025
 U 1 1 5915EFD1
 P 10150 3150
-F 0 "#PWR029" H 10150 2900 50  0001 C CNN
+F 0 "#PWR025" H 10150 2900 50  0001 C CNN
 F 1 "GND" H 10150 3000 50  0000 C CNN
 F 2 "" H 10150 3150 50  0000 C CNN
@@
 	10350 3900 10150 3900
 $Comp
-L GND #PWR030
+L GND #PWR026
 U 1 1 5915F857
 P 10150 3950
-F 0 "#PWR030" H 10150 3700 50  0001 C CNN
+F 0 "#PWR026" H 10150 3700 50  0001 C CNN
 F 1 "GND" H 10150 3800 50  0000 C CNN
 F 2 "" H 10150 3950 50  0000 C CNN
@@
 	10350 4700 10150 4700
 $Comp
-L GND #PWR031
+L GND #PWR027
 U 1 1 5915FBD1
 P 10150 4750
-F 0 "#PWR031" H 10150 4500 50  0001 C CNN
+F 0 "#PWR027" H 10150 4500 50  0001 C CNN
 F 1 "GND" H 10150 4600 50  0000 C CNN
 F 2 "" H 10150 4750 50  0000 C CNN
@@
 	10150 5500 10150 5550
 $Comp
-L GND #PWR032
+L GND #PWR028
 U 1 1 59160C14
 P 10150 5550
-F 0 "#PWR032" H 10150 5300 50  0001 C CNN
+F 0 "#PWR028" H 10150 5300 50  0001 C CNN
 F 1 "GND" H 10150 5400 50  0000 C CNN
 F 2 "" H 10150 5550 50  0000 C CNN
@@
 $EndComp
 $Comp
-L GND #PWR033
+L GND #PWR029
 U 1 1 59165506
 P 7900 2600
-F 0 "#PWR033" H 7900 2350 50  0001 C CNN
+F 0 "#PWR029" H 7900 2350 50  0001 C CNN
 F 1 "GND" H 7900 2450 50  0000 C CNN
 F 2 "" H 7900 2600 50  0000 C CNN
@@
 	7900 2550 7900 2600
 $Comp
-L GND #PWR034
+L GND #PWR030
 U 1 1 59165674
 P 7900 2050
-F 0 "#PWR034" H 7900 1800 50  0001 C CNN
+F 0 "#PWR030" H 7900 1800 50  0001 C CNN
 F 1 "GND" H 7900 1900 50  0000 C CNN
 F 2 "" H 7900 2050 50  0000 C CNN
@@
 	7650 3150 7650 3200
 $Comp
-L GND #PWR035
+L GND #PWR031
 U 1 1 59165F7C
 P 7650 3200
-F 0 "#PWR035" H 7650 2950 50  0001 C CNN
+F 0 "#PWR031" H 7650 2950 50  0001 C CNN
 F 1 "GND" H 7650 3050 50  0000 C CNN
 F 2 "" H 7650 3200 50  0000 C CNN
@@
 Text Label 7450 2450 2    60   ~ 0
 LED
+NoConn ~ 2900 1500
+NoConn ~ 2100 1500
+NoConn ~ 3500 5400
+NoConn ~ 3500 5500
 $EndSCHEMATC

Commit message: Started PCB layout
Parts:
- added W1, W2, W3, W4: TEST_1P, Mounting_Holes:MountingHole_3.2mm_M3_Pad, symbol TEST_1P
Connections:
- net GND: now also W1.1, W2.1, W3.1, W4.1
Changed lines of the file:
@@
 NoConn ~ 3500 5400
 NoConn ~ 3500 5500
+$Comp
+L TEST_1P W1
+U 1 1 5918C302
+P 1300 6900
+F 0 "W1" H 1300 7170 50  0000 C CNN
+F 1 "TEST_1P" H 1300 7100 50  0000 C CNN
+F 2 "Mounting_Holes:MountingHole_3.2mm_M3_Pad" H 1500 6900 50  0001 C CNN
+F 3 "" H 1500 6900 50  0000 C CNN
+	1    1300 6900
+	1    0    0    -1
+$EndComp
+$Comp
+L TEST_1P W2
+U 1 1 5918C82F
+P 1650 6900
+F 0 "W2" H 1650 7170 50  0000 C CNN
+F 1 "TEST_1P" H 1650 7100 50  0000 C CNN
+F 2 "Mounting_Holes:MountingHole_3.2mm_M3_Pad" H 1850 6900 50  0001 C CNN
+F 3 "" H 1850 6900 50  0000 C CNN
+	1    1650 6900
+	1    0    0    -1
+$EndComp
+$Comp
+L TEST_1P W3
+U 1 1 5918C8B3
+P 2000 6900
+F 0 "W3" H 2000 7170 50  0000 C CNN
+F 1 "TEST_1P" H 2000 7100 50  0000 C CNN
+F 2 "Mounting_Holes:MountingHole_3.2mm_M3_Pad" H 2200 6900 50  0001 C CNN
+F 3 "" H 2200 6900 50  0000 C CNN
+	1    2000 6900
+	1    0    0    -1
+$EndComp
+$Comp
+L TEST_1P W4
+U 1 1 5918C936
+P 2350 6900
+F 0 "W4" H 2350 7170 50  0000 C CNN
+F 1 "TEST_1P" H 2350 7100 50  0000 C CNN
+F 2 "Mounting_Holes:MountingHole_3.2mm_M3_Pad" H 2550 6900 50  0001 C CNN
+F 3 "" H 2550 6900 50  0000 C CNN
+	1    2350 6900
+	1    0    0    -1
+$EndComp
+$Comp
+L GND #PWR?
+U 1 1 5918CADC
+P 1300 6950
+F 0 "#PWR?" H 1300 6700 50  0001 C CNN
+F 1 "GND" H 1300 6800 50  0000 C CNN
+F 2 "" H 1300 6950 50  0000 C CNN
+F 3 "" H 1300 6950 50  0000 C CNN
+	1    1300 6950
+	1    0    0    -1
+$EndComp
+$Comp
+L GND #PWR?
+U 1 1 5918CB53
+P 1650 6950
+F 0 "#PWR?" H 1650 6700 50  0001 C CNN
+F 1 "GND" H 1650 6800 50  0000 C CNN
+F 2 "" H 1650 6950 50  0000 C CNN
+F 3 "" H 1650 6950 50  0000 C CNN
+	1    1650 6950
+	1    0    0    -1
+$EndComp
+$Comp
+L GND #PWR?
+U 1 1 5918CBCA
+P 2000 6950
+F 0 "#PWR?" H 2000 6700 50  0001 C CNN
+F 1 "GND" H 2000 6800 50  0000 C CNN
+F 2 "" H 2000 6950 50  0000 C CNN
+F 3 "" H 2000 6950 50  0000 C CNN
+	1    2000 6950
+	1    0    0    -1
+$EndComp
+$Comp
+L GND #PWR?
+U 1 1 5918CC41
+P 2350 6950
+F 0 "#PWR?" H 2350 6700 50  0001 C CNN
+F 1 "GND" H 2350 6800 50  0000 C CNN
+F 2 "" H 2350 6950 50  0000 C CNN
+F 3 "" H 2350 6950 50  0000 C CNN
+	1    2350 6950
+	1    0    0    -1
+$EndComp
+Wire Wire Line
+	2350 6900 2350 6950
+Wire Wire Line
+	2000 6900 2000 6950
+Wire Wire Line
+	1650 6900 1650 6950
+Wire Wire Line
+	1300 6900 1300 6950
 $EndSCHEMATC

Commit message: 30x50mm board
Parts:
- J2: footprint kuro:4x2_1.27mm_SMD_header -> Pin_Headers:Pin_Header_Straight_2x04_Pitch2.54mm
Changed lines of the file:
@@
 F 0 "J2" H 6350 4100 50  0000 C CNN
 F 1 "CONN_02X04" H 6350 3600 50  0000 C CNN
-F 2 "kuro:4x2_1.27mm_SMD_header" H 6350 2650 50  0001 C CNN
+F 2 "Pin_Headers:Pin_Header_Straight_2x04_Pitch2.54mm" H 6350 2650 50  0001 C CNN
 F 3 "" H 6350 2650 50  0000 C CNN
 	1    6350 3850
